File: IOB-RR-CirKits_array.brd (EAGLE design)
At the start: 104.1 x 106.7 mm, 25 parts

Commit message: normalized silkscreen layout across IOBs
Parts:
- added FID-UL, FID_LR: FIDUCIAL, SPCoast:FIDUCIAL_1MM
- FID1X11, FID1X12, FID2X11, FID2X12: value (none) -> FIDUCIAL
- JP1X11, JP1X12: value (none) -> CONNECTOR-M05X2PTH
- R10X11, R10X12, R11X11, R11X12, R12X11, R12X12, R1X11, R1X12, R2X11, R2X12, R3X11, R3X12, R4X11, R4X12, R9X11, R9X12: value (none) -> NOSTUFF
- U$1X11, U$1X12: value (none) -> IO4-IOB-DUALRR-CIRKITS
Routing:
- net GNDX12: track 26.7 -> 0.00 mm
- net GNDX11: track 26.7 -> 0.00 mm
- added copper zone on layer 1, net VCCX11
- added copper zone on layer 1, net VCCX12
Other:
- board text added: "1.0"
- board text added: "JP1"
- board text added: "R1"
- board text added: "R10"
- board text added: "R11"
- board text added: "R12"
- board text added: "R2"
- board text added: "R3"
- board text added: "R4"
- board text added: "R9"
- board text added: "Yellow Headers"
- board text added: "Yellow Soldermask White Silkscreen"
- board text added: "^ Cut if using resistors v"
- board text removed: "Yellow Soldermask Black Silkscreen"
- board text removed: "^ Cut if adding resistors"
- board text removed: "v1.0"
